Commit message: Add dae files

File: cpp_impl/src/edubot/urdf/robot.urdf (robot description, URDF)
Before this commit: robot robot, 7 links, 6 joints
Links:
- link base: geometry collision cylinder length=${base_height} radius=${base_radius}; visual mesh filename=package://edubot/meshes/Base.dae scale=1 1 1
- link link1: geometry collision box size=${link_width} ${link_height} ${link_1_length}; visual mesh filename=package://edubot/meshes/Link1.dae scale=1 1 1
- link link2: geometry collision box size=${link_width} ${link_height} ${link_2_length}; visual mesh filename=package://edubot/meshes/Link2.dae scale=1 1 1
- link link3: geometry collision box size=${link_width} ${link_height} ${link_3_length}; visual mesh filename=package://edubot/meshes/Link3.dae scale=1 1 1
- link link4: geometry collision box size=${link_width} ${link_height} ${link_4_length}; visual mesh filename=package://edubot/meshes/Link4.dae scale=1 1 1
Joints:
- joint link2_joint: axis 1 0 0 -> 0 1 0
- joint link3_joint: axis 1 0 0 -> 0 1 0
- joint link4_joint: axis 1 0 0 -> 0 1 0

Commit message: Add movable gripper to edubot

File: cpp_impl/src/edubot/urdf/robot.urdf (robot description, URDF)
Before this commit: robot robot, 7 links, 6 joints
Links:
- added link gripper_left; collision box size=${link_width/2} ${link_height/4} ${link_4_length/2}; visual mesh filename=package://edubot/meshes/GripperLeft.dae scale=1 1 1
- added link gripper_right; collision box size=${link_width/2} ${link_height/4} ${link_4_length/2}; visual mesh filename=package://edubot/meshes/GripperRight.dae scale=1 1 1
Joints:
- added joint gripper_left_joint: type prismatic, parent ee, child gripper_left, origin xyz=0 -0.01 -0.025 rpy=0 0 0, axis 0 1 0, limit lower=${-0.0} upper=${0.02} effort=10 velocity=10
- added joint gripper_right_joint: type prismatic, parent ee, child gripper_right, origin xyz=0 0.01 -0.025 rpy=0 0 0, axis 0 1 0, limit lower=${-0.0} upper=${0.02} effort=10 velocity=10, mimic joint=gripper_left_joint multiplier=-1 offset=0

Commit message: Synchronized hardware specifications

File: cpp_impl/src/edubot/urdf/robot.urdf (robot description, URDF)
Before this commit: robot robot, 9 links, 8 joints
Joints:
- joint link2_joint: origin xyz=0 0 ${link_1_length} rpy=0 0 0 -> xyz=0 0 ${link_1_length} rpy=0 ${-PI_2} 0
- joint link3_joint: origin xyz=0 0 ${link_2_length} rpy=0 0 0 -> xyz=0 0 ${link_2_length} rpy=0 ${PI_2} 0
- joint link4_joint: origin xyz=0 0 ${link_3_length} rpy=0 0 0 -> xyz=0 0 ${link_3_length} rpy=0 ${-PI_2} 0

Commit message: Fix error in rad2ticks and urdf misalignment

File: cpp_impl/src/edubot/urdf/robot.urdf (robot description, URDF)
Before this commit: robot robot, 9 links, 8 joints
Joints:
- joint link2_joint: origin xyz=0 0 ${link_1_length} rpy=0 ${-PI_2} 0 -> xyz=0 0 ${link_1_length} rpy=0 0 0
- joint link3_joint: origin xyz=0 0 ${link_2_length} rpy=0 ${PI_2} 0 -> xyz=0 0 ${link_2_length} rpy=0 ${PI_2} ${PI}
- joint link4_joint: origin xyz=0 0 ${link_3_length} rpy=0 ${-PI_2} 0 -> xyz=0 0 ${link_3_length} rpy=0 0 ${-PI}
